File: smartWinder-ESP/schematic/smartWinder-ESP.sch (KiCad schematic (older format))
At the start: 39 parts, among them IC2 MP2315GJ-Z, J1 Conn_01x09, J2 Conn_01x06, U1 LTV-847S, U2 ESP-12E

Commit message: Added VIN Sensing to the PCB
Parts:
- removed TP3: TestPoint, TestPoint:TestPoint_Pad_D1.0mm, symbol Connector:TestPoint
- added C12: 100nF, Capacitor_SMD:C_0805_2012Metric_Pad1.15x1.40mm_HandSolder, symbol Device:C_Small
- added R18: 430k, Resistor_SMD:R_0805_2012Metric_Pad1.15x1.40mm_HandSolder, symbol Device:R_Small
- added R19: 10k, Resistor_SMD:R_0805_2012Metric_Pad1.15x1.40mm_HandSolder, symbol Device:R_Small
- J1: footprint Connector_PinSocket_2.54mm:PinSocket_1x09_P2.54mm_Vertical -> Connector_PinHeader_2.54mm:PinHeader_1x09_P2.54mm_Vertical
- renumbered TP4 to TP3, TP5 to TP4
Connections:
- net +24V: now also R18.1
- net GND: now also C12.2, R19.2
- net at U2.2 (ADC): now also C12.1, R18.2, R19.1
Changed lines of the file:
@@
 	7600 5800 7600 5750
-$Comp
-L Connector:TestPoint TP3
-U 1 1 5DA65A46
-P 6350 4650
-F 0 "TP3" V 6545 4722 50  0000 C CNN
-F 1 "TestPoint" V 6454 4722 50  0000 C CNN
-F 2 "TestPoint:TestPoint_Pad_D1.0mm" H 6550 4650 50  0001 C CNN
-F 3 "~" H 6550 4650 50  0001 C CNN
-	1    6350 4650
-	0    -1   -1   0
-$EndComp
-Wire Wire Line
-	6350 4650 6600 4650
 $Comp
 L Device:R_Small R13
@@
 F 0 "J1" H 1818 5867 50  0000 C CNN
 F 1 "Conn_01x09" H 1818 5776 50  0000 C CNN
-F 2 "Connector_PinSocket_2.54mm:PinSocket_1x09_P2.54mm_Vertical" H 1900 5250 50  0001 C CNN
+F 2 "Connector_PinHeader_2.54mm:PinHeader_1x09_P2.54mm_Vertical" H 1900 5250 50  0001 C CNN
 F 3 "~" H 1900 5250 50  0001 C CNN
 	1    1900 5250
@@
 IMPULS2
 $Comp
-L Connector:TestPoint TP4
+L Connector:TestPoint TP3
 U 1 1 5DCF2EED
 P 8350 4850
-F 0 "TP4" V 8545 4922 50  0000 C CNN
+F 0 "TP3" V 8545 4922 50  0000 C CNN
 F 1 "TestPoint" V 8454 4922 50  0000 C CNN
 F 2 "TestPoint:TestPoint_Pad_D1.0mm" H 8550 4850 50  0001 C CNN
@@
 $EndComp
 $Comp
-L Connector:TestPoint TP5
+L Connector:TestPoint TP4
 U 1 1 5DCF3DD6
 P 8350 5250
-F 0 "TP5" V 8545 5322 50  0000 C CNN
+F 0 "TP4" V 8545 5322 50  0000 C CNN
 F 1 "TestPoint" V 8454 5322 50  0000 C CNN
 F 2 "TestPoint:TestPoint_Pad_D1.0mm" H 8550 5250 50  0001 C CNN
@@
 Wire Wire Line
 	6950 1750 6950 1950
+$Comp
+L Device:R_Small R18
+U 1 1 5DB6298D
+P 5700 4500
+F 0 "R18" H 5759 4546 50  0000 L CNN
+F 1 "430k" H 5759 4455 50  0000 L CNN
+F 2 "Resistor_SMD:R_0805_2012Metric_Pad1.15x1.40mm_HandSolder" H 5700 4500 50  0001 C CNN
+F 3 "~" H 5700 4500 50  0001 C CNN
+	1    5700 4500
+	1    0    0    -1
+$EndComp
+$Comp
+L Device:R_Small R19
+U 1 1 5DB63307
+P 5700 4800
+F 0 "R19" H 5759 4846 50  0000 L CNN
+F 1 "10k" H 5759 4755 50  0000 L CNN
+F 2 "Resistor_SMD:R_0805_2012Metric_Pad1.15x1.40mm_HandSolder" H 5700 4800 50  0001 C CNN
+F 3 "~" H 5700 4800 50  0001 C CNN
+	1    5700 4800
+	1    0    0    -1
+$EndComp
+Wire Wire Line
+	5700 4650 5700 4600
+Wire Wire Line
+	5700 4650 6050 4650
+Wire Wire Line
+	5700 4650 5700 4700
+Connection ~ 5700 4650
+Wire Wire Line
+	5700 4400 5700 4350
+Wire Wire Line
+	5700 4900 5700 4950
+$Comp
+L power:GND #PWR0101
+U 1 1 5DB7E4B9
+P 5700 4950
+F 0 "#PWR0101" H 5700 4700 50  0001 C CNN
+F 1 "GND" H 5705 4777 50  0000 C CNN
+F 2 "" H 5700 4950 50  0001 C CNN
+F 3 "" H 5700 4950 50  0001 C CNN
+	1    5700 4950
+	1    0    0    -1
+$EndComp
+$Comp
+L power:+24V #PWR0118
+U 1 1 5DB7F6DA
+P 5700 4350
+F 0 "#PWR0118" H 5700 4200 50  0001 C CNN
+F 1 "+24V" H 5715 4523 50  0000 C CNN
+F 2 "" H 5700 4350 50  0001 C CNN
+F 3 "" H 5700 4350 50  0001 C CNN
+	1    5700 4350
+	1    0    0    -1
+$EndComp
+$Comp
+L Device:C_Small C12
+U 1 1 5DB9405E
+P 6050 4800
+F 0 "C12" H 6142 4846 50  0000 L CNN
+F 1 "100nF" H 6142 4755 50  0000 L CNN
+F 2 "Capacitor_SMD:C_0805_2012Metric_Pad1.15x1.40mm_HandSolder" H 6050 4800 50  0001 C CNN
+F 3 "~" H 6050 4800 50  0001 C CNN
+	1    6050 4800
+	1    0    0    -1
+$EndComp
+$Comp
+L power:GND #PWR0119
+U 1 1 5DB94A5C
+P 6050 4950
+F 0 "#PWR0119" H 6050 4700 50  0001 C CNN
+F 1 "GND" H 6055 4777 50  0000 C CNN
+F 2 "" H 6050 4950 50  0001 C CNN
+F 3 "" H 6050 4950 50  0001 C CNN
+	1    6050 4950
+	1    0    0    -1
+$EndComp
+Wire Wire Line
+	6050 4950 6050 4900
+Wire Wire Line
+	6050 4700 6050 4650
+Connection ~ 6050 4650
+Wire Wire Line
+	6050 4650 6600 4650
 $EndSCHEMATC

Commit message: Finalized PCB and sent to Production
Finalized PCB and sent to Production
Generated PDF and 3D PCB File
Parts:
- R10: value 10 k -> 10k
- R13, R14, R15, R16, R17: value 12k -> 10k
- renumbered TP2 to 3V3, TP1 to GND1, TP3 to IO12, TP4 to IO16
Other:
- moved on the sheet: J2
Changed lines of the file:
@@
 EESchema Schematic File Version 4
+LIBS:smartWinder-ESP-cache
 EELAYER 30 0
 EELAYER END
@@
 P 2650 5450
 F 0 "R10" H 2709 5496 50  0000 L CNN
-F 1 "10 k" H 2709 5405 50  0000 L CNN
+F 1 "10k" H 2709 5405 50  0000 L CNN
 F 2 "Resistor_SMD:R_0805_2012Metric_Pad1.15x1.40mm_HandSolder" H 2650 5450 50  0001 C CNN
 F 3 "~" H 2650 5450 50  0001 C CNN
@@
 P 9600 4450
 F 0 "R13" H 9659 4496 50  0000 L CNN
-F 1 "12k" H 9659 4405 50  0000 L CNN
+F 1 "10k" H 9659 4405 50  0000 L CNN
 F 2 "Resistor_SMD:R_0805_2012Metric_Pad1.15x1.40mm_HandSolder" H 9600 4450 50  0001 C CNN
 F 3 "~" H 9600 4450 50  0001 C CNN
@@
 P 9600 4700
 F 0 "R14" H 9659 4746 50  0000 L CNN
-F 1 "12k" H 9659 4655 50  0000 L CNN
+F 1 "10k" H 9659 4655 50  0000 L CNN
 F 2 "Resistor_SMD:R_0805_2012Metric_Pad1.15x1.40mm_HandSolder" H 9600 4700 50  0001 C CNN
 F 3 "~" H 9600 4700 50  0001 C CNN
@@
 P 9600 4950
 F 0 "R15" H 9659 4996 50  0000 L CNN
-F 1 "12k" H 9659 4905 50  0000 L CNN
+F 1 "10k" H 9659 4905 50  0000 L CNN
 F 2 "Resistor_SMD:R_0805_2012Metric_Pad1.15x1.40mm_HandSolder" H 9600 4950 50  0001 C CNN
 F 3 "~" H 9600 4950 50  0001 C CNN
@@
 P 9600 5200
 F 0 "R16" H 9659 5246 50  0000 L CNN
-F 1 "12k" H 9659 5155 50  0000 L CNN
+F 1 "10k" H 9659 5155 50  0000 L CNN
 F 2 "Resistor_SMD:R_0805_2012Metric_Pad1.15x1.40mm_HandSolder" H 9600 5200 50  0001 C CNN
 F 3 "~" H 9600 5200 50  0001 C CNN
@@
 P 9600 5600
 F 0 "R17" H 9659 5646 50  0000 L CNN
-F 1 "12k" H 9659 5555 50  0000 L CNN
+F 1 "10k" H 9659 5555 50  0000 L CNN
 F 2 "Resistor_SMD:R_0805_2012Metric_Pad1.15x1.40mm_HandSolder" H 9600 5600 50  0001 C CNN
 F 3 "~" H 9600 5600 50  0001 C CNN
@@
 L Connector_Generic:Conn_01x06 J2
 U 1 1 5DA7C0BE
-P 10450 2250
-F 0 "J2" H 10250 2700 50  0000 L CNN
-F 1 "Conn_01x06" H 10050 2600 50  0000 L CNN
-F 2 "Connector_PinHeader_2.54mm:PinHeader_1x06_P2.54mm_Vertical" H 10450 2250 50  0001 C CNN
-F 3 "~" H 10450 2250 50  0001 C CNN
-	1    10450 2250
+P 9900 2100
+F 0 "J2" H 9700 2550 50  0000 L CNN
+F 1 "Conn_01x06" H 9500 2450 50  0000 L CNN
+F 2 "Connector_PinHeader_2.54mm:PinHeader_1x06_P2.54mm_Vertical" H 9900 2100 50  0001 C CNN
+F 3 "~" H 9900 2100 50  0001 C CNN
+	1    9900 2100
 	1    0    0    -1
 $EndComp
@@
 L power:GND #PWR0116
 U 1 1 5DA83DB2
-P 10150 2050
-F 0 "#PWR0116" H 10150 1800 50  0001 C CNN
-F 1 "GND" V 10155 1922 50  0000 R CNN
-F 2 "" H 10150 2050 50  0001 C CNN
-F 3 "" H 10150 2050 50  0001 C CNN
-	1    10150 2050
+P 9600 1900
+F 0 "#PWR0116" H 9600 1650 50  0001 C CNN
+F 1 "GND" V 9605 1772 50  0000 R CNN
+F 2 "" H 9600 1900 50  0001 C CNN
+F 3 "" H 9600 1900 50  0001 C CNN
+	1    9600 1900
 	0    1    1    0
 $EndComp
@@
 L power:+3V3 #PWR0117
 U 1 1 5DA855FB
-P 10150 2350
-F 0 "#PWR0117" H 10150 2200 50  0001 C CNN
-F 1 "+3V3" V 10165 2478 50  0000 L CNN
-F 2 "" H 10150 2350 50  0001 C CNN
-F 3 "" H 10150 2350 50  0001 C CNN
-	1    10150 2350
-	0    -1   -1   0
-$EndComp
-Wire Wire Line
-	10150 2050 10250 2050
-Wire Wire Line
-	9600 2150 10250 2150
-Wire Wire Line
-	10250 2250 9600 2250
-Wire Wire Line
-	10250 2350 10150 2350
-Wire Wire Line
-	10250 2450 9600 2450
-Wire Wire Line
-	10250 2550 9600 2550
-Text Label 9600 2150 0    50   ~ 0
+P 9600 2200
+F 0 "#PWR0117" H 9600 2050 50  0001 C CNN
+F 1 "+3V3" V 9615 2328 50  0000 L CNN
+F 2 "" H 9600 2200 50  0001 C CNN
+F 3 "" H 9600 2200 50  0001 C CNN
+	1    9600 2200
+	0    -1   -1   0
+$EndComp
+Wire Wire Line
+	9600 1900 9700 1900
+Wire Wire Line
+	9050 2000 9700 2000
+Wire Wire Line
+	9700 2100 9050 2100
+Wire Wire Line
+	9700 2200 9600 2200
+Wire Wire Line
+	9700 2300 9050 2300
+Wire Wire Line
+	9700 2400 9050 2400
+Text Label 9050 2000 0    50   ~ 0
 TXD
-Text Label 9600 2250 0    50   ~ 0
+Text Label 9050 2100 0    50   ~ 0
 RXD
-Text Label 9600 2450 0    50   ~ 0
+Text Label 9050 2300 0    50   ~ 0
 GPIO0
-Text Label 9600 2550 0    50   ~ 0
+Text Label 9050 2400 0    50   ~ 0
 RST
 Text Notes 2950 4650 2    50   ~ 0
@@
 IMPULS2
 $Comp
-L Connector:TestPoint TP3
+L Connector:TestPoint IO12
 U 1 1 5DCF2EED
 P 8350 4850
-F 0 "TP3" V 8545 4922 50  0000 C CNN
+F 0 "IO12" V 8545 4922 50  0000 C CNN
 F 1 "TestPoint" V 8454 4922 50  0000 C CNN
 F 2 "TestPoint:TestPoint_Pad_D1.0mm" H 8550 4850 50  0001 C CNN
@@
 $EndComp
 $Comp
-L Connector:TestPoint TP4
+L Connector:TestPoint IO16
 U 1 1 5DCF3DD6
 P 8350 5250
-F 0 "TP4" V 8545 5322 50  0000 C CNN
+F 0 "IO16" V 8545 5322 50  0000 C CNN
 F 1 "TestPoint" V 8454 5322 50  0000 C CNN
 F 2 "TestPoint:TestPoint_Pad_D1.0mm" H 8550 5250 50  0001 C CNN
@@
 ESP8266
 $Comp
-L Connector:TestPoint TP2
-U 1 1 5DBCBDC9
-P 7150 1950
-F 0 "TP2" V 7345 2022 50  0000 C CNN
-F 1 "TestPoint" V 7254 2022 50  0000 C CNN
-F 2 "TestPoint:TestPoint_Pad_D1.0mm" H 7350 1950 50  0001 C CNN
-F 3 "~" H 7350 1950 50  0001 C CNN
-	1    7150 1950
-	0    1    -1   0
-$EndComp
-$Comp
-L Connector:TestPoint TP1
+L Connector:TestPoint GND1
 U 1 1 5DBCC763
 P 7150 2050
-F 0 "TP1" V 7345 2122 50  0000 C CNN
+F 0 "GND1" V 7345 2122 50  0000 C CNN
 F 1 "TestPoint" V 7254 2122 50  0000 C CNN
 F 2 "TestPoint:TestPoint_Pad_D1.0mm" H 7350 2050 50  0001 C CNN
@@
 Wire Wire Line
 	6050 4650 6600 4650
+$Comp
+L Connector:TestPoint 3V3
+U 1 1 5DBCBDC9
+P 7150 1950
+F 0 "3V3" V 7345 2022 50  0000 C CNN
+F 1 "TestPoint" V 7254 2022 50  0000 C CNN
+F 2 "TestPoint:TestPoint_Pad_D1.0mm" H 7350 1950 50  0001 C CNN
+F 3 "~" H 7350 1950 50  0001 C CNN
+	1    7150 1950
+	0    1    -1   0
+$EndComp
 $EndSCHEMATC
